File: hardware/OpenRX-Gemini.kicad_pcb (KiCad board)
At the start: 6 copper layers, 57.6 x 16 mm, 194 parts, among them T1 0900PC16J0042001E, T4 0900PC16J0042001E, T5 0900PC16J0042001E, U1 ESP32-C3FH4, U1 OW7EL89CENUYO3YLC-32M, U15 RFX2401C, U16 SKY13414-485LF, U17 RFX2401C, U18 SKY13414-485LF, U2 LR1121IMLTRT, U2 TLV75533PDQNR, U3 ESP32-C3FH4, U3 SX1281IMLTRT, U3 TS2306A 240GF MSM 9_C2976675, U4 LR1121IMLTRT, U4 TS2306A 240GF MSM 9_C2976675, U5 OW7EL89CENUYO3YLC-32M, U6 TLV75533PDQNR, U7 RFX2401C, U8 SKY13414-485LF, U9 LR1121IMLTRT, X1 CJ17-400001010B20

Commit message: gemini initial
Parts:
- removed the AE1 at (94.9, 47.0)
- removed the AE1 at (70.3, 44.4)
- removed the AE1 at (115.6, 51.6)
- removed the AE1 at (102.0, 51.6)
- removed AE2: 47948-0001, OpenRX-Shared:ANT-SMD_47948-0001
- removed the C1 at (91.5, 46.7)
- removed the C1 at (77.5, 48.6)
- removed the C1 at (104.1, 52.7)
- removed the C1 at (117.7, 52.7)
- removed the C10 at (69.1, 50.7)
- removed the C10 at (108.2, 52.6)
- removed the C10 at (121.8, 52.6)
- removed the C11 at (73.3, 47.3)
- removed the C11 at (108.0, 47.2)
- removed the C11 at (121.6, 47.2)
- removed the C11 at (95.2, 55.5)
- removed the C12 at (79.7, 48.4)
- removed the C12 at (104.6, 45.1)
- removed the C12 at (118.2, 45.1)
- removed the C12 at (92.9, 56.2)
- removed the C13 at (103.5, 53.3)
- removed the C13 at (117.2, 53.5)
- removed the C13 at (69.8, 56.0)
- removed the C13 at (94.2, 55.0)
- removed the C14 at (116.1, 50.5)
- removed the C14 at (102.5, 49.9)
- removed the C14 at (80.0, 56.0)
- removed the C14 at (89.6, 48.8)
- removed the C15 at (69.1, 49.5)
- removed the C15 at (90.0, 44.3)
- removed the C15 at (120.7, 53.4)
- removed the C15 at (107.1, 53.4)
- removed the C16 at (77.6, 52.8)
- removed the C16 at (87.9, 44.3)
- removed the C16 at (105.8, 53.6)
- removed the C16 at (119.4, 53.6)
- removed the C17 at (122.1, 51.6)
- removed the C17 at (73.3, 46.8)
- removed the C17 at (108.5, 51.6)
- removed the C18 at (122.1, 52.9)
- removed the C18 at (93.0, 44.8)
- removed the C18 at (108.5, 52.9)
- removed the C18 at (69.2, 48.1)
- removed the C19 at (94.1, 49.6)
- removed the C19 at (102.5, 51.0)
- removed the C19 at (116.1, 51.2)
- removed the C2 at (91.5, 47.3)
- removed the C2 at (70.7, 47.3)
- removed the C2 at (115.5, 46.7)
- removed the C2 at (101.9, 46.7)
- removed the C20 at (116.1, 49.8)
- removed the C20 at (79.7, 53.2)
- removed the C20 at (102.5, 49.4)
- removed the C20 at (92.9, 49.3)
- removed the C22 at (79.8, 52.4)
- removed the C22 at (91.8, 56.3)
- removed the C24 at (80.8, 50.8)
- removed the C24 at (88.4, 56.3)
- removed the C3 at (86.9, 53.0)
- removed the C3 at (77.3, 47.6)
- removed the C3 at (106.8, 52.0)
- removed the C3 at (120.4, 52.0)
- removed the C4 at (76.0, 50.7)
- removed the C4 at (87.8, 56.3)
- removed the C4 at (117.1, 52.7)
- removed the C4 at (103.5, 52.7)
- removed C45: 0.3pF, Capacitor_SMD:C_0201_0603Metric
- removed C46: 220pF, Capacitor_SMD:C_0201_0603Metric
- removed C47: 1uF, Capacitor_SMD:C_0201_0603Metric
- removed the C5 at (87.0, 49.6)
- removed the C5 at (116.2, 48.7)
- removed the C5 at (102.6, 48.7)
- removed the C6 at (95.1, 49.9)
- removed the C6 at (76.6, 48.2)
- removed the C6 at (115.6, 48.7)
- removed the C6 at (102.0, 48.7)
- removed the C7 at (107.0, 45.4)
- removed the C7 at (120.6, 45.4)
- removed the C7 at (94.1, 52.5)
- removed the C7 at (73.0, 56.1)
- removed the C8 at (88.7, 47.0)
- removed the C8 at (76.3, 52.5)
- removed the C8 at (121.6, 51.8)
- removed the C8 at (108.0, 51.8)
- removed the C9 at (108.7, 47.2)
- removed the C9 at (122.3, 47.2)
- removed the C9 at (94.0, 56.7)
- removed the C9 at (75.1, 48.9)
- removed the D1 at (108.2, 45.4)
- removed the D1 at (80.7, 48.4)
- removed the D1 at (91.8, 44.8)
- removed the D1 at (121.7, 45.4)
- removed the FL1 at (118.6, 47.9)
- removed the FL1 at (105.0, 47.9)
- removed the FL1 at (88.4, 48.9)
- removed FL4, FL5: 2450FM07D0034T, OpenRX-Shared:FILTER-SMD_4P-L1.0-W0.5-L
- removed JP1 (x2), JP4, JP5: U.FL-R-SMT-1(80), OpenRX-Shared:RF-SMD_FRF05002-JSS103M
- removed the L1 at (76.6, 48.7)
- removed the L1 at (90.1, 56.4)
- removed the L1 at (117.4, 51.7)
- removed the L1 at (103.8, 51.7)
- removed the L2 at (94.1, 50.3)
- removed the L2 at (71.4, 56.1)
- removed the OSC1 at (102.2, 52.6)
- removed the OSC1 at (115.7, 52.9)
- removed the R1 at (70.7, 46.7)
- removed the R1 at (89.3, 47.0)
- removed the R1 at (102.5, 46.7)
- removed the R1 at (116.0, 46.7)
- removed the R2 at (71.6, 47.0)
- removed the R2 at (115.8, 47.7)
- removed the R2 at (87.1, 49.5)
- removed the R2 at (102.3, 47.7)
- removed the R3 at (86.9, 51.8)
- removed the R3 at (76.9, 52.5)
- removed the R3 at (119.6, 45.1)
- removed the R3 at (106.0, 45.1)
- removed the R4 at (72.3, 47.0)
- removed the R4 at (89.8, 47.0)
- removed the R4 at (107.9, 45.1)
- removed the R4 at (121.5, 45.1)
- removed the R5 at (87.0, 51.2)
- removed the R5 at (74.9, 55.9)
- removed the R6 at (68.8, 52.1)
- removed the R6 at (94.2, 54.4)
- removed T4, T5: 0900PC16J0042001E, OpenRX-Shared:FILTER-SMD_10P-L2.0-W1.6-BL
- removed the TP1 at (115.3, 55.5)
- removed the TP1 at (101.8, 55.5)
- removed the TP1 at (71.5, 55.8)
- removed the TP1 at (87.4, 56.6)
- removed the TP2 at (104.0, 55.5)
- removed the TP2 at (117.5, 55.5)
- removed the TP2 at (74.1, 55.8)
- removed the TP2 at (90.0, 56.6)
- removed the TP3 at (76.6, 55.8)
- removed the TP3 at (108.4, 55.5)
- removed the TP3 at (92.5, 56.6)
- removed the TP3 at (121.9, 55.5)
- removed the TP4 at (119.7, 55.5)
- removed the TP4 at (79.1, 55.8)
- removed the TP4 at (106.2, 55.5)
- removed the TP4 at (95.1, 56.6)
- removed TP5: Boot, OpenRX-Shared:SolderPad_1.2x2.0mm
- removed TP5 (x2): GND, OpenRX-Shared:SolderPad_1.2x2.0mm
- removed the U1 at (78.6, 50.3)
- removed the U1 at (90.1, 50.6)
- removed the U1 at (119.4, 48.4)
- removed the U1 at (105.9, 48.4)
- removed U15, U17: RFX2401C, OpenRX-Shared:QFN-16_L3.0-W3.0-P0.50-BL-EP1.7
- removed U16, U18: SKY13414-485LF, OpenRX-Shared:QFN-14_L2.0-W2.0-P0.45-BL-EP
- removed the U2 at (94.1, 55.8)
- removed the U2 at (121.8, 53.5)
- removed the U2 at (108.2, 53.5)
- removed the U2 at (72.3, 52.5)
- removed the U3 at (105.7, 51.2)
- removed the U3 at (119.3, 51.2)
- removed the U3 at (72.3, 50.5)
- removed the U3 at (88.7, 45.0)
- removed the U4 at (69.3, 55.0)
- removed the U4 at (90.3, 52.5)
- removed the X1 at (94.4, 51.4)
- removed the X1 at (76.3, 49.7)
- removed the X1 at (119.0, 52.2)
- removed the X1 at (105.5, 52.2)
- added AE1: 2450AT18A100E, OpenRX-Shared:ANT-SMD_L3.2-W1.6, B.Cu at (115.9, 112.0)
- added C1: 15pF, Capacitor_SMD:C_0201_0603Metric, B.Cu at (114.2, 112.2)
- added C10: 1uF, Capacitor_SMD:C_0201_0603Metric, B.Cu at (100.7, 111.4)
- added C11: 10uF, Capacitor_SMD:C_0402_1005Metric, F.Cu at (107.6, 114.5)
- added C12: 100nF, Capacitor_SMD:C_0201_0603Metric, F.Cu at (115.4, 101.2)
- added C13: 100nF, Capacitor_SMD:C_0201_0603Metric, F.Cu at (108.4, 110.0)
- added C14: 100nF, Capacitor_SMD:C_0201_0603Metric, F.Cu at (100.8, 109.0)
- added C15: 47pF, Capacitor_SMD:C_0201_0603Metric, F.Cu at (100.8, 109.7)
- added C16: 100nF, Capacitor_SMD:C_0201_0603Metric, B.Cu at (104.8, 112.2)
- added C17: 1uF, Capacitor_SMD:C_0201_0603Metric, B.Cu at (101.7, 110.2)
- added C18: 10uF, Capacitor_SMD:C_0402_1005Metric, B.Cu at (101.8, 109.3)
- added C19: 2.2nF, Capacitor_SMD:C_0201_0603Metric, F.Cu at (101.2, 108.3)
- added C2: 47p, Capacitor_SMD:C_0201_0603Metric, F.Cu at (100.8, 107.2)
- added C20: 470nF, Capacitor_SMD:C_0201_0603Metric, F.Cu at (105.0, 114.2)
- added C22: 1n, Capacitor_SMD:C_0201_0603Metric, B.Cu at (105.0, 102.8)
- added C24: 47p, Capacitor_SMD:C_0201_0603Metric, F.Cu at (102.5, 103.3)
- added C3: 15pF, Capacitor_SMD:C_0201_0603Metric, B.Cu at (114.2, 109.7)
- added C30: 1.2pF, Capacitor_SMD:C_0201_0603Metric, B.Cu at (111.3, 116.0)
- added C31: 1uF, Capacitor_SMD:C_0201_0603Metric, B.Cu at (106.4, 104.9)
- added C33: 2.2nF, Capacitor_SMD:C_0201_0603Metric, F.Cu at (109.8, 110.0)
- added C34: 10pF, Capacitor_SMD:C_0201_0603Metric, F.Cu at (108.0, 113.4)
- added C35: 100nF, Capacitor_SMD:C_0201_0603Metric, B.Cu at (112.8, 110.9)
- added C36: 47pF, Capacitor_SMD:C_0201_0603Metric, B.Cu at (112.8, 111.6)
- added C37: 100nF, Capacitor_SMD:C_0201_0603Metric, F.Cu at (115.2, 115.9)
- added C38: 470nF, Capacitor_SMD:C_0201_0603Metric, F.Cu at (113.1, 115.9)
- added C39: 47p, Capacitor_SMD:C_0201_0603Metric, F.Cu at (108.7, 108.8)
- added C4: 1uF, Capacitor_SMD:C_0201_0603Metric, B.Cu at (112.8, 112.3)
- added C40: 220pF, Capacitor_SMD:C_0201_0603Metric, B.Cu at (114.0, 106.3)
- added C41: 1uF, Capacitor_SMD:C_0201_0603Metric, B.Cu at (114.0, 105.6)
- added C5: 100nF, Capacitor_SMD:C_0201_0603Metric, B.Cu at (105.5, 112.2)
- added C6: 100nF, Capacitor_SMD:C_0201_0603Metric, B.Cu at (106.8, 107.7)
- added C7: 10pF, Capacitor_SMD:C_0201_0603Metric, F.Cu at (101.2, 112.5)
- added C8: 10uF, Capacitor_SMD:C_0402_1005Metric, B.Cu at (101.2, 112.6)
- added C9: 100nF, Capacitor_SMD:C_0201_0603Metric, B.Cu at (106.8, 114.7)
- added D1: XL-1010RGBC-WS2812B, OpenRX-Shared:LED-SMD_4P-L1.0-W1.0-TL_XL-1010RGBC-WS2812B, F.Cu at (114.2, 101.2)
- added FL1: 2450FM07D0034T, OpenRX-Shared:FILTER-SMD_4P-L1.0-W0.5-L, F.Cu at (107.0, 107.2)
- added FL2: 2450FM07D0034T, OpenRX-Shared:FILTER-SMD_4P-L1.0-W0.5-L, F.Cu at (115.0, 108.4)
- added J1: Conn_Coaxial_Small, Connector_Coaxial:U.FL_Hirose_U.FL-R-SMT-1_Vertical, F.Cu at (102.2, 100.7)
- added J2: Conn_Coaxial_Small, Connector_Coaxial:U.FL_Hirose_U.FL-R-SMT-1_Vertical, F.Cu at (110.0, 100.7)
- added L1: 10uH, Inductor_SMD:L_0603_1608Metric, B.Cu at (104.7, 114.0)
- added L2: 24nH, Inductor_SMD:L_0201_0603Metric, B.Cu at (114.2, 113.0)
- added L4: 2.5nH, Inductor_SMD:L_0201_0603Metric, B.Cu at (110.7, 115.6)
- added L5: 47nH, Inductor_SMD:L_0402_1005Metric, F.Cu at (102.2, 106.8)
- added L6: 10uH, Inductor_SMD:L_0603_1608Metric, B.Cu at (113.5, 115.2)
- added L7: 47nH, Inductor_SMD:L_0402_1005Metric, F.Cu at (110.0, 108.5)
- added OSC1: OW7EL89CENUYO3YLC-32M, OpenRX-Shared:OSC-SMD_4P-L2.0-W1.6-BL_TXC_7Z, F.Cu at (108.8, 111.7)
- added R1: 200, Resistor_SMD:R_0201_0603Metric, F.Cu at (102.0, 106.0)
- added R12: 100k, Resistor_SMD:R_0201_0603Metric, F.Cu at (116.6, 103.3)
- added R2: 10k, Resistor_SMD:R_0201_0603Metric, B.Cu at (101.0, 114.2)
- added R3: 10k, Resistor_SMD:R_0201_0603Metric, B.Cu at (105.2, 111.2)
- added R4: 10k, Resistor_SMD:R_0201_0603Metric, B.Cu at (116.2, 106.5)
- added R5: 10k, Resistor_SMD:R_0201_0603Metric, B.Cu at (102.2, 114.0)
- added R6: 220, Resistor_SMD:R_0201_0603Metric, F.Cu at (101.2, 111.2)
- added T2: 0900PC16J0042001E, OpenRX-Shared:FILTER-SMD_10P-L2.0-W1.6-BL, F.Cu at (112.0, 107.7)
- added TP1: RX, OpenRX-Shared:SolderPad_1.2x2.0mm, F.Cu at (101.3, 117.0)
- added TP2: TX, OpenRX-Shared:SolderPad_1.2x2.0mm, F.Cu at (103.8, 117.0)
- added TP3: 5V, OpenRX-Shared:SolderPad_1.2x2.0mm, F.Cu at (106.4, 117.0)
- added TP4: GND, OpenRX-Shared:SolderPad_1.2x2.0mm, F.Cu at (108.9, 117.0)
- added U1: ESP32-C3, Package_DFN_QFN:QFN-32-1EP_5x5mm_P0.5mm_EP3.7x3.7mm, B.Cu at (109.0, 111.1)
- added U2: TLV75533PDQNR, OpenRX-Shared:X2SON-4_L1.0-W1.0-P0.65-TL-EP, B.Cu at (101.7, 111.3)
- added U3: LR1121IMLTRT, Package_DFN_QFN:QFN-32-1EP_5x5mm_P0.5mm_EP3.7x3.7mm, F.Cu at (104.6, 110.8)
- added U4: RFX2401C, OpenRX-Shared:QFN-16_L3.0-W3.0-P0.50-BL-EP1.7, F.Cu at (107.5, 104.9)
- added X1: CJ17-400001010B20, OpenRX-Shared:CRYSTAL-SMD_4P-L1.6-W1.2-BL, B.Cu at (114.2, 111.0)
- C21: value 100nF -> 220pF
- C23: value 100nF -> 47p; moved to F.Cu
- C25: value 100nF -> 1uF; moved to B.Cu
- C26: value 100nF -> 10nF
- C27: value 10pF -> 1uF; moved to B.Cu
- C28: value 4.7uF -> 1uF; footprint Capacitor_SMD:C_0402_1005Metric -> Capacitor_SMD:C_0201_0603Metric
- C29: value 100nF -> 1.2pF
- C42: value 0.3pF -> 47p; moved to F.Cu
- C43: value 220pF -> 1n
- C44: value 1uF -> 47p; moved to F.Cu
- L3: value 10uH -> 2.0nH; footprint Inductor_SMD:L_0603_1608Metric -> Inductor_SMD:L_0201_0603Metric
- R10: value 680R -> 200
- R11, R7: value 10k -> 100k
- R8: value 220R -> 100k
- R9: value 680R -> 220; moved to F.Cu
- T1, U7: moved to F.Cu
- U5: value OW7EL89CENUYO3YLC-32M -> SKY13373-460LF; footprint OpenRX-Shared:OSC-SMD_4P-L2.0-W1.6-BL_TXC_7Z -> OpenRX-Shared:QFN-12_EP_2x2_Pitch0.5mm; moved to F.Cu
- U6: value TLV75533PDQNR -> LR1121IMLTRT; footprint OpenRX-Shared:X2SON-4_L1.0-W1.0-P0.65-TL-EP -> Package_DFN_QFN:QFN-32-1EP_5x5mm_P0.5mm_EP3.7x3.7mm
- U8: value SKY13414-485LF -> SKY13373-460LF; footprint OpenRX-Shared:QFN-14_L2.0-W2.0-P0.45-BL-EP -> OpenRX-Shared:QFN-12_EP_2x2_Pitch0.5mm; moved to F.Cu
- U9: value LR1121IMLTRT -> TS2306A 240GF MSM 9_C2976675; footprint OpenRX-Shared:QFN-32_L5.0-W5.0-P0.50-BL-EP3.7 -> OpenRX-Shared:SW-SMD_4P-L3.0-W2.0-P0.85-LS3.5
- moved R11 76.8 mm to (116.6, 107.8)
- moved R9 75.4 mm to (109.4, 113.4), turned to 0 degrees
- moved C42 73.3 mm to (113.7, 103.2)
- moved C44 70.4 mm to (110.0, 103.5), turned to 90 degrees
- moved C28 70.4 mm to (102.8, 114.0), turned to -90 degrees
- moved C25 70.2 mm to (109.6, 114.5), turned to 0 degrees
- moved C43 69.3 mm to (112.5, 104.4), turned to 180 degrees
- moved U6 69.1 mm to (113.2, 112.5), turned to 0 degrees
- moved C29 68.5 mm to (111.0, 114.5), turned to 0 degrees
- moved R7 67.9 mm to (109.3, 106.8), turned to 180 degrees
- moved U9 66.4 mm to (114.9, 108.0), turned to 180 degrees
- moved C26 66.3 mm to (112.8, 113.0), turned to 0 degrees
- moved L3 66.2 mm to (108.2, 114.5)
- moved R10 64.9 mm to (109.8, 107.7), turned to 0 degrees
- moved U7 64.8 mm to (115.0, 105.5), turned to 0 degrees
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Connections:
- C23 pad 1: GND -> Net-(U4-ANT)
- C23 pad 2: Net-(U4-VTCXO) -> Net-(U5-J2)
- C25 pad 1: GND -> Net-(C25-Pad1)
- C25 pad 2: /ESP32-C3 + 2x LR1121 Gemini/VTCXO -> GND
- C26 pad 1: GND -> +3V3
- C26 pad 2: Net-(U9-VREG) -> GND
- C27 pad 1: Net-(C27-Pad1) -> +3V3
- C27 pad 2: Net-(U9-XTA) -> GND
- C28 pad 1: Net-(U9-VR_PA) -> /ESP32-C3/CHIP_EN
- C29 pad 1: GND -> Net-(U1-LNA_IN)
- C29 pad 2: +3V3 -> GND
- C42 pad 1: Net-(U15-ANT) -> Net-(U7-ANT)
- C42 pad 2: GND -> Net-(U8-J2)
- C44 pad 1: +3V3 -> Net-(U8-RFC)
- C44 pad 2: GND -> Net-(J2-In)
- L3 pad 1: Net-(U9-DCC_SW) -> Net-(C25-Pad1)
- R10 pad 1: Net-(U9-DIO4) -> /LR1121_B/VR_PA
- R10 pad 2: /ESP32-C3 + 2x LR1121 Gemini/MISO -> Net-(T2-RFO_HP_LF)
- R11 pad 1: +3V3 -> GND
- R11 pad 2: /ESP32-C3 + 2x LR1121 Gemini/BUSY2 -> /LR1121_B/TXEN24
- R7 pad 1: +3V3 -> GND
- R7 pad 2: /ESP32-C3 + 2x LR1121 Gemini/BUTTON -> /LR1121_A/TXEN24
- R8 pad 1: Net-(C27-Pad1) -> +3V3
- R8 pad 2: /ESP32-C3 + 2x LR1121 Gemini/XTA -> /LR1121_A/RXEN24
- R9 pad 2: /ESP32-C3 + 2x LR1121 Gemini/MISO -> Net-(U6-XTA)
- U5 pad 1: GND -> Net-(T1-TX_HP)
- U5 pad 3: Net-(U5-OUTPUT) -> Net-(T1-RX)
- U5 pad 4: Net-(U4-VTCXO) -> /LR1121_A/CTRL1
- U6 pad 1: +3V3 -> /LR1121_B/VR_PA
- U6 pad 2: GND -> +3V3
- U6 pad 3: +5V -> /Clock/VTCXO
- U6 pad 4: +5V -> Net-(U6-XTA)
- U6 pad 5: GND -> unconnected-(U6-XTB-Pad5)
- U7 pad 14: +3V3 -> unconnected-(U7-VDD-Pad14)
- U7 pad 5: /ESP32-C3 + LR1121 Mono/TXEN -> /LR1121_B/TXEN24
- U7 pad 6: /ESP32-C3 + LR1121 Mono/RXEN -> /LR1121_B/RXEN24
- U8 pad 10: Net-(U7-ANT) -> GND
- U8 pad 11: unconnected-(U8-N/C-Pad11) -> Net-(U8-RFC)
- U8 pad 12: unconnected-(U8-N/C-Pad12) -> GND
- U8 pad 13: Net-(JP1-SIG) -> GND
- U8 pad 2: Net-(T1-TX_HP) -> GND
- U8 pad 3: Net-(T1-RX) -> Net-(T2-RX)
- U8 pad 4: +3V3 -> /LR1121_B/CTRL1
- U8 pad 5: /ESP32-C3 + LR1121 Mono/DIO7-1 -> /LR1121_B/CTRL2
- U8 pad 6: /ESP32-C3 + LR1121 Mono/DIO8-1 -> +3V3
- U8 pad 9: unconnected-(U8-RF2-Pad9) -> Net-(U8-J2)
- U9 pad 1: Net-(U9-VR_PA) -> /ESP32-C3/BOOT
- U9 pad 2: +3V3 -> GND
Routing:
- net GND: track 298.1 -> 21.7 mm, vias 220 -> 42
- net +3V3: track 121.9 -> 13.0 mm, vias 42 -> 11
- net +5V: track 66.8 -> 11.0 mm, vias 12 -> 2
- net Net-(U1-U0RXD): track 32.2 -> 0.99 mm, vias 4 -> 1
- net Net-(U1-U0TXD): track 29.5 -> 3.64 mm, vias 2 -> 1
- net /ESP32-C3 + LR1121 Mono/BUTTON: track 18.2 -> 0.00 mm
- net /ESP32-C3 + 2x LR1121 Gemini/RST1: track 14.5 -> 0.00 mm, vias 2 -> 0
- net /ESP32-C3 + 2x LR1121 Gemini/DIO8-1: track 14.2 -> 0.00 mm, vias 2 -> 0
- net /ESP32-C3 + SX1281 Core/RST: track 13.2 -> 0.00 mm, vias 1 -> 0
- net /ESP32-C3 + 2x LR1121 Gemini/DIO7-2: track 13.0 -> 0.00 mm, vias 2 -> 0
- net /ESP32-C3 + 2x LR1121 Gemini/IRQ1: track 12.9 -> 0.00 mm, vias 2 -> 0
- net /ESP32-C3 + LR1121 Mono/LED: track 12.0 -> 0.00 mm, vias 2 -> 0
- net /ESP32-C3 + SX1281 Core (UFL)/RST: track 11.8 -> 0.00 mm, vias 1 -> 0
- net /Clock/TCXO_Out: track 0.00 -> 11.6 mm, vias 0 -> 2
- net /ESP32-C3 + 2x LR1121 Gemini/DIO8-2: track 11.6 -> 0.00 mm, vias 2 -> 0
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- added copper zone on B.Cu, net +3V3
- added copper zone on B.Cu, net +5V
- removed copper zone on In2.Cu, net +3V3
- removed copper zone on In3.Cu, net +3V3
- removed copper zone on B.Cu, net GND
- removed copper zone on F.Cu, net GND
- removed copper zone on In1.Cu, net GND
- removed copper zone on In2.Cu, net GND
- removed copper zone on In3.Cu, net GND
- removed copper zone on In4.Cu, net GND
Other:
- board size 57.6 x 16 mm -> 17 x 17.6 mm
- board text added: "5V"
- board text removed: "-"
- board text removed: "5v"
- board text removed: "boot"
- board text removed: "open"
- board text removed: "rx"
- board text removed: "tx"
