File: hardware/esp32-c3.kicad_sch (KiCad schematic)
At the start: 36 parts, among them U1 ESP32-C3, U2 TLV75533PDQNR, U9 TS2306A 240GF MSM 9_C2976675, X1 CJ17-400001010B20

Commit message: Give every placed part an LCSC field
The BOM exporter reads a field named LCSC. Parts that carried only
"LCSC Part" were dropped from the supplier BOM and the pick and place
without a warning, and ESP32-C3, the 15uH DC-DC inductor and
SKY13373-460LF carried no LCSC anywhere.

Adds LCSC to the schematic symbols and mirrors it onto the board
footprints, which is the only route for references created by a
replicated hierarchical sheet. Numbers verified against the LCSC
catalogue: ESP32-C3FH4 C2858491, MLZ2012M150WT000 C383402,
SKY13373-460LF C150853. Bare test pads stay without a part number.

Co-Authored-By: Claude Opus 5 (1M context) <noreply@anthropic.com>
Claude-Session: https://claude.ai/code/session_01HXA6SP2VEuBZn7yMrez3es
Parts:
- U1: LCSC (none) -> C2858491; MPN (none) -> ESP32-C3FH4; Manufacturer (none) -> Espressif Systems
